File: CST simulation/First Wilkinson PD/Wilkinson PD.kicad_pcb (KiCad board)
At the start: 2 copper layers, 6 parts

Commit message: new s
Parts:
- removed R1: 102, Resistor_SMD:R_0402_1005Metric
- removed R2: 176, Resistor_SMD:R_0402_1005Metric
- renumbered U3 to U1, U1 to U3
Connections:
- WPD1 pad 4: Net-(R1-Pad1) -> unconnected-(WPD1-R1-Pad4)
- WPD1 pad 5: Net-(R1-Pad2) -> unconnected-(WPD1-R1-Pad5)
- WPD1 pad 6: Net-(R2-Pad1) -> unconnected-(WPD1-R2-Pad6)
- WPD1 pad 7: Net-(R2-Pad2) -> unconnected-(WPD1-R2-Pad7)
Other:
- board outline added: 36.5 x 17 mm
