File: CST simulation/SecondWilkinson PD/Wilkinson PD.kicad_pcb (KiCad board)
At the start: 2 copper layers, 4 parts

Commit message: new wpd
Parts:
- moved U2 3.91 mm to (171.5, 89.7)
- moved U3 3.91 mm to (171.5, 77.5)
Changed lines of the file:
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@@
 	(footprint "RF_WPD:Pad for termination"
 		(layer "F.Cu")
-		(at 169 86.7336)
+		(at 171.5 89.7336)
 		(property "Reference" "U2"
 			(at 0 -0.5 0)
@@
 	(footprint "RF_WPD:Pad for termination"
 		(layer "F.Cu")
-		(at 169 80.5)
+		(at 171.5 77.5)
 		(property "Reference" "U3"
 			(at 0 -0.5 0)
@@
 	)
 	(gr_line
+		(start 164.48024 84.5312)
+		(end 167.5 89.7336)
+		(stroke
+			(width 1.06426)
+			(type solid)
+		)
+		(layer "F.Cu")
+		(net 1)
+	)
+	(gr_line
 		(start 164.48024 82.7024)
-		(end 166.4716 80.5)
+		(end 167.5 77.5)
 		(stroke
 			(width 1.06426)
@@
 	)
 	(gr_line
-		(start 166.4716 86.7336)
-		(end 169 86.7336)
+		(start 167.5 89.7336)
+		(end 171.5 89.7336)
 		(stroke
 			(width 1.06426)
@@
 	)
 	(gr_line
-		(start 166.4716 80.5)
-		(end 169 80.5)
+		(start 167.5 77.5)
+		(end 171.5 77.5)
 		(stroke
 			(width 1.06426)
@@
 		(layer "F.Cu")
 		(net 2)
-	)
-	(gr_line
-		(start 164.48024 84.5312)
-		(end 166.4716 86.7336)
-		(stroke
-			(width 1.06426)
-			(type solid)
-		)
-		(layer "F.Cu")
-		(net 1)
 	)
 	(segment
@@
 		(net 3)
 	)
+	(group ""
+		(members "557a3f6d-b076-4cd7-a99d-5e2783ec98bd" "b6b57ee7-4b3d-49a1-9119-b5e52bc48871")
+	)
+	(group ""
+		(members "96c36a85-d9be-4808-826a-a5d6649ecb80" "fd0c0a27-3109-4b70-8402-416a644a0e6f")
+	)
 	(embedded_fonts no)
