File: CST simulation/SecondWilkinson PD/test/test.kicad_pcb (KiCad board)
At the start: 2 copper layers, 2 parts

Commit message: wpd_test3
Parts:
- removed JP1: Jumper_2_Bridged, JumperWires:Jumper-Wire_12mm_Red
- removed R1: R, Resistor_SMD:R_0201_0603Metric
- added U1: ~, PDG Footprints:WPD_Input_Output_Pad, F.Cu at (180.2, 76.8)
- added U2: ~, PDG Footprints:WPD_Input_Output_Pad, F.Cu at (216.9, 66.2)
- added U3: ~, PDG Footprints:WPD_Input_Output_Pad, F.Cu at (216.9, 89.9)
- added WPD1: ~, PDG Footprints:WPD_2Ring_10500_RO4350B_test3, F.Cu at (193.3, 76.9)
Routing:
- net Net-(U3-port2): track 0.00 -> 24.5 mm
- net Net-(U2-port2): track 0.00 -> 24.5 mm
- net Net-(U1-port1): track 0.00 -> 10.5 mm
