File: CST simulation/SecondWilkinson PD/test/test.kicad_sch (KiCad schematic)
At the start: 0 parts

Commit message: paper
Parts:
- added JP1: Jumper_2_Bridged, JumperWires:Jumper-Wire_12mm_Red, symbol Jumper:Jumper_2_Bridged
- added R1: R, Resistor_SMD:R_0201_0603Metric, symbol Device:R
Connections:
- new net: JP1.2 (B), R1.1
- new net +4V: JP1.1 (A)
- new net GND: R1.2

Commit message: wpd_test3
Parts:
- removed JP1: Jumper_2_Bridged, JumperWires:Jumper-Wire_12mm_Red, symbol Jumper:Jumper_2_Bridged
- removed R1: R, Resistor_SMD:R_0201_0603Metric, symbol Device:R
- added U1: ~, PDG Footprints:WPD_Input_Output_Pad, symbol PDG:Port
- added U2, U3: ~, PDG Footprints:WPD_Input_Output_Pad, symbol PDG:port2
- added WPD1: ~, PDG Footprints:WPD_2Ring_10500_RO4350B_test3, symbol PDG:WPD_2Ring
Connections:
- new net: U3.1 (port2), WPD1.3 (PD2)
- new net: U1.1 (port1), WPD1.1 (In)
- new net: U2.1 (port2), WPD1.2 (PD1)
